File: PCB/RH2288_PWM.kicad_pcb (KiCad board)
At the start: 2 copper layers, 15.2 x 29.2 mm, 9 parts, among them J2 AVR_ICSP, J3 Conn_FANs, J4 Conn_RH2288_V2, J5 UART, U1 78L05_SOT23, U2 ATmega328P-MMH

Commit message: PCB finished
Parts:
- moved R1 5.88 mm to (152.6, 92.1), turned to 180 degrees
Connections:
- J3 pad 2: Net-(J3-Pad2) -> FAN_SEN1
- J3 pad 4: Net-(J3-Pad4) -> FAN_PWM
- J3 pad 5: Net-(J3-Pad5) -> FAN_SEN2
- J4 pad 2: Net-(J4-Pad2) -> PWM_OUT
- J4 pad 4: Net-(J4-Pad4) -> PWM_IN
- J4 pad 5: Net-(J4-Pad5) -> PWM_OUT
- J5 pad 2: TXD -> FAN_SEN1
- U2 pad 1: Net-(U2-Pad1) -> PWM_OUT
- U2 pad 11: Net-(U2-Pad11) -> FAN_SEN2
- U2 pad 12: Net-(U2-Pad12) -> FAN_PWM
- U2 pad 27: TXD -> FAN_SEN1
- U2 pad 6: Net-(U2-Pad6) -> PWM_IN
Routing:
- net FAN_SEN1: track 0.00 -> 19.1 mm
- net PWM_OUT: track 0.00 -> 14.6 mm
- net FAN_PWM: track 0.00 -> 11.9 mm
- net FAN_SEN2: track 0.00 -> 11.6 mm
- net GND: track 1.64 -> 9.72 mm
- net PWM_IN: track 0.00 -> 7.25 mm, vias 0 -> 1
- net +5V: track 23.4 -> 29.0 mm, vias 3 -> 4
- net TXD: track 4.83 -> 0.00 mm
- added copper zone on F.Cu, net GND
Other:
- rule pad_to_mask_clearance: 0.051 -> 0.0508
